File: hw/hydrasucrela/FPGA_3.kicad_sch (KiCad schematic)
At the start: 9 parts, among them Q2 Q_NPN_BCE, U1 ECP5U_25_CABGA381, U2 ECP5U_25_CABGA381, U5 XUY73, U6 MCP23S08-E/SO

Commit message: hw: update kicad footprints and symbols
Parts:
- removed Q2: Q_NPN_BCE, symbol Device:Q_NPN_BCE
- added Q1: MMBTA06, Package_TO_SOT_SMD:SOT-23, symbol Transistor_BJT:MMBTA06
- C6: footprint (none) -> Capacitor_SMD:C_0603_1608Metric_Pad1.08x0.95mm_HandSolder
- R4, R5, R6: footprint (none) -> Resistor_SMD:R_0603_1608Metric_Pad0.98x0.95mm_HandSolder
- U1: footprint (none) -> Package_BGA:Lattice_caBGA-381_17.0x17.0mm_Layout20x20_P0.8mm_Ball0.4mm_Pad0.4mm_NSMD
- renumbered U2 to U1
Connections:
- net GND: now also Q1.2 (E)
- net SCS0: now also Q1.1 (B)
- net at R6.2, U6.7 (CS): now also Q1.3 (C)
Changed lines of the file:
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@@
 	)
 	(junction
-		(at 83.82 176.53)
-		(diameter 0)
-		(color 0 0 0 0)
-	)
-	(junction
 		(at 99.06 184.15)
 		(diameter 0)
@@
 	)
 	(junction
+		(at 83.82 176.53)
+		(diameter 0)
+		(color 0 0 0 0)
+	)
+	(junction
 		(at 111.76 156.21)
 		(diameter 0)
@@
 	)
 	(symbol
-		(lib_id "Device:Q_NPN_BCE")
-		(at 81.28 181.61 0)
-		(unit 1)
-		(exclude_from_sim no)
-		(in_bom yes)
-		(on_board yes)
-		(dnp no)
-		(fields_autoplaced yes)
-		(property "Reference" "Q2"
-			(at 86.36 180.3399 0)
-			(effects
-				(font
-					(size 1.27 1.27)
-				)
-				(justify left)
-			)
-		)
-		(property "Value" "Q_NPN_BCE"
-			(at 86.36 182.8799 0)
-			(effects
-				(font
-					(size 1.27 1.27)
-				)
-				(justify left)
-			)
-		)
-		(property "Footprint" ""
-			(at 86.36 179.07 0)
-			(effects
-				(font
-					(size 1.27 1.27)
-				)
-				(hide yes)
-			)
-		)
-		(property "Datasheet" "~"
-			(at 81.28 181.61 0)
-			(effects
-				(font
-					(size 1.27 1.27)
-				)
-				(hide yes)
-			)
-		)
-		(property "Description" "NPN transistor, base/collector/emitter"
-			(at 81.28 181.61 0)
-			(effects
-				(font
-					(size 1.27 1.27)
-				)
-				(hide yes)
-			)
-		)
-		(pin "1"
-		)
-		(pin "2"
-		)
-		(pin "3"
-		)
-		(instances
-			(project ""
-				(path "/7dca55fc-548f-4319-89ea-8fc153556669/76f71ab5-50fa-4de0-b0e9-cddae93b7c4d"
-					(reference "Q2")
-					(unit 1)
-				)
-			)
-		)
-	)
-	(symbol
 		(lib_id "Lattice_ECP5_FPGA:ECP5U_25_CABGA381")
 		(at 153.67 140.97 0)
@@
 			)
 		)
-		(property "Footprint" ""
+		(property "Footprint" "Package_BGA:Lattice_caBGA-381_17.0x17.0mm_Layout20x20_P0.8mm_Ball0.4mm_Pad0.4mm_NSMD"
 			(at 157.48 139.7 0)
 			(effects
@@
 			)
 		)
-		(property "Footprint" ""
+		(property "Footprint" "Resistor_SMD:R_0603_1608Metric_Pad0.98x0.95mm_HandSolder"
 			(at 141.732 57.15 90)
 			(effects
@@
 			)
 		)
-		(property "Footprint" ""
+		(property "Footprint" "Resistor_SMD:R_0603_1608Metric_Pad0.98x0.95mm_HandSolder"
 			(at 82.042 172.72 90)
 			(effects
@@
 			)
 		)
-		(property "Footprint" ""
+		(property "Footprint" "Capacitor_SMD:C_0603_1608Metric_Pad1.08x0.95mm_HandSolder"
 			(at 25.7048 172.72 0)
 			(effects
@@
 			)
 		)
-		(property "Footprint" ""
+		(property "Footprint" "Package_BGA:Lattice_caBGA-381_17.0x17.0mm_Layout20x20_P0.8mm_Ball0.4mm_Pad0.4mm_NSMD"
 			(at 62.23 58.42 0)
 			(effects
@@
 		(dnp no)
 		(fields_autoplaced yes)
-		(property "Reference" "U2"
+		(property "Reference" "U1"
 			(at 208.28 73.6599 0)
 			(effects
@@
 			(project "hydrasucrela"
 				(path "/7dca55fc-548f-4319-89ea-8fc153556669/76f71ab5-50fa-4de0-b0e9-cddae93b7c4d"
-					(reference "U2")
+					(reference "U1")
 					(unit 8)
 				)
@@
 			)
 		)
-		(property "Footprint" ""
+		(property "Footprint" "Resistor_SMD:R_0603_1608Metric_Pad0.98x0.95mm_HandSolder"
 			(at 140.462 88.9 90)
 			(effects
@@
 					(unit 1)
 				)
+			)
+		)
+	)
+	(symbol
+		(lib_id "Transistor_BJT:MMBTA06")
+		(at 81.28 181.61 0)
+		(unit 1)
+		(exclude_from_sim no)
+		(in_bom yes)
+		(on_board yes)
+		(dnp no)
+		(fields_autoplaced yes)
+		(property "Reference" "Q1"
+			(at 86.36 180.3399 0)
+			(effects
+				(font
+					(size 1.27 1.27)
+				)
+				(justify left)
+			)
+		)
+		(property "Value" "MMBTA06"
+			(at 86.36 182.8799 0)
+			(effects
+				(font
+					(size 1.27 1.27)
+				)
+				(justify left)
+			)
+		)
+		(property "Footprint" "Package_TO_SOT_SMD:SOT-23"
+			(at 86.36 183.515 0)
+			(effects
+				(font
+					(size 1.27 1.27)
+					(italic yes)
+				)
+				(justify left)
+				(hide yes)
+			)
+		)
+		(property "Datasheet" "https://diotec.com/request/datasheet/mmbta06.pdf"
+			(at 81.28 181.61 0)
+			(effects
+				(font
+					(size 1.27 1.27)
+				)
+				(justify left)
+				(hide yes)
+			)
+		)
+		(property "Description" "0.5A Ic, 80V Vce, general purpose NPN"
+			(at 81.28 181.61 0)
+			(effects
+				(font
+					(size 1.27 1.27)
+				)
+				(hide yes)
+			)
+		)
+		(pin "3"
+		)
+		(pin "1"
+		)
+		(pin "2"
+		)
+		(instances
+			(project ""
+				(path "/7dca55fc-548f-4319-89ea-8fc153556669/76f71ab5-50fa-4de0-b0e9-cddae93b7c4d"
+					(reference "Q1")
+					(unit 1)
+				)

Commit message: Update HydraSucreLA PCB
Connections:
- net Probe_10 is gone; now on net Probe_4: U1.C1 (PL17A/+/HS/LDQ20)
- net Probe_7 is gone; now on net Probe_6: U1.E3 (PL11B/-/HS/LDQ8)
- net Probe_8 is gone; now on net Probe_0: U1.A2 (PL14A/+/HS/LDQ20)
- net Probe_9 is gone; now on net Probe_2: U1.B1 (PL14B/-/HS/LDQ20)
- net Probe_0: no longer U1.A4 (PL2A/+/HS/LDQ8)
- net Probe_1: now also U1.A4 (PL2A/+/HS/LDQ8); no longer U1.A5 (PL2B/-/HS/LDQ8)
- net Probe_2: no longer U1.C4 (PL5A/+/HS/LDQ8)
- net Probe_4: no longer U1.E4 (PL8A/+/HS/LDQS8)
- net Probe_5: now also U1.C4 (PL5A/+/HS/LDQ8); no longer U1.D5 (PL8B/-/HS/LDQSN8)
- net Probe_6: no longer U1.F4 (PL11A/+/HS/LDQ8)
- net RXD_1: now reaches U1.R1 (PB4A/+/D7/IO7)
- net TXD_1: now reaches U1.T1 (PB4B/-/D6/IO6)
- net Probe_11: no longer names the net of U1.D1 (PL17B/-/HS/LDQ20)
- net Probe_12: no longer names the net of U1.H4 (PL20A/+/GR_PCLK7_1/HS/LDQS20)
- net Probe_13: no longer names the net of U1.G5 (PL20B/-/HS/LDQSN20)
- net Probe_14: no longer names the net of U1.G3 (PL23A/+/PCLKT7_1/HS/LDQ20)
- net Probe_15: no longer names the net of U1.F3 (PL23B/-/PCLKC7_1/HS/LDQ20)
- no-connect marks 33 -> 40
